Commit message: Add x, y, angle and its velocities in plugin feedback

File: spherorobot_cpp/urdf/vibro_table.urdf (robot description, URDF)
Before this commit: robot vibro_table, 3 links, 2 joints
Joints:
- joint left_rail_joint: origin xyz=0 0.045 0.001 rpy=0 0 0 -> xyz=0 0.04 0.001 rpy=0 0 0
- joint right_rail_joint: origin xyz=0 -0.045 0.001 rpy=0 0 0 -> xyz=0 -0.04 0.001 rpy=0 0 0
